File: eeprom-lc_12_2/eeprom-lc_12_2.kicad_sch (KiCad schematic)
At the start: 9 parts

Commit message: Some work on eeprom code and pcb
Parts:
- removed Data_EEPROM: TXS0108EPW, Package_SO:TSSOP-20_4.4x6.5mm_P0.65mm, symbol Logic_LevelTranslator:TXS0108EPW
- added J1: Conn_02x05_Pin, Connector_PinHeader_2.00mm:PinHeader_2x05_P2.00mm_Vertical, symbol Connector:Conn_01x10_Pin
- CONTROLLER_P2040, EEPROM_RP2040: footprint WeAct-rp2040:WeAct-RP2040-Pico -> WeAct-RP2040-Pico:WeAct-RP2040-Pico; symbol WeAct-rp2040:WeAct-RP2040-Pico -> WeAct-RP2040-Pico:WeAct-RP2040-Pico
- WIFI-ESP32C6: value MOUDLE-SEEEDUINO-XIAO -> WeAct-RP2040-Pico; footprint XIAO-rp2040:MOUDLE14P-2.54-21X17.8MM -> XIAO_PCB:MOUDLE14P-2.54-21X17.8MM; symbol XIAO-rp2040:MOUDLE-SEEEDUINO-XIAO -> MOUDLE-SEEEDUINO-XIAO:MOUDLE-SEEEDUINO-XIAO
- renumbered Data_Controller to Data_Lines1
Connections:
- net A0_3V3: no longer CONTROLLER_P2040.2 (GP1)
- net A10_3V3: no longer CONTROLLER_P2040.13 (GP11)
- net A11_3V3: no longer CONTROLLER_P2040.14 (GP12)
- net A12_3V3: no longer CONTROLLER_P2040.16 (GP13)
- net A13_3V3: no longer CONTROLLER_P2040.17 (GP14)
- net A14_3V3: no longer CONTROLLER_P2040.18 (GP15)
- net A15_3V3: no longer CONTROLLER_P2040.19 (GP16)
- net A16_3V3: no longer CONTROLLER_P2040.20 (GP17)
- net A1_3V3: no longer CONTROLLER_P2040.3 (GP2)
- net A2_3V3: no longer CONTROLLER_P2040.4 (GP3)
- net A3_3V3: no longer CONTROLLER_P2040.5 (GP4)
- net A4_3V3: no longer CONTROLLER_P2040.7 (GP5)
- net A5_3V3: no longer CONTROLLER_P2040.8 (GP6)
- net A6_3V3: no longer CONTROLLER_P2040.9 (GP7)
- net A7_3V3: no longer CONTROLLER_P2040.10 (GP8)
- net A8_3V3: no longer CONTROLLER_P2040.11 (GP9)
- net A9_3V3: no longer CONTROLLER_P2040.12 (GP10)
- net GND: now also CONTROLLER_P2040.38 (GND), EEPROM_RP2040.38 (GND), J1.10 (Pin_10); no longer CONTROLLER_P2040.15 (GND), CONTROLLER_P2040.6 (GND), EEPROM_RP2040.15 (GND), EEPROM_RP2040.6 (GND), EEPROM_SLOT1.24 (~G)
- net OE_3V3: no longer CONTROLLER_P2040.1 (GP0), EEPROM_RP2040.1 (GP0)
- net VCC_3V3: now also Address_0_7.10 (OE), Address_16_OE1.10 (OE), Address_8_15.10 (OE), CONTROLLER_P2040.36 (3V3), Data_Lines1.10 (OE), EEPROM_RP2040.36 (3V3), WIFI-ESP32C6.12 (3V3)
- net VCC_5V: now also CONTROLLER_P2040.39 (VIN), EEPROM_RP2040.39 (VIN); no longer EEPROM_SLOT1.1 (VPP), EEPROM_SLOT1.31 (~P)
- net D0_3V3: now reaches EEPROM_RP2040.21 (GP18)
- net D0_3V3: now also Data_Lines1.1 (A1)
- net D1_3V3: now reaches EEPROM_RP2040.22 (GP19)
- net D1_3V3: now also Data_Lines1.3 (A2)
- net D2_3V3: now reaches EEPROM_RP2040.23 (GP20)
- net D2_3V3: now also Data_Lines1.4 (A3)
- net D3_3V3: now reaches EEPROM_RP2040.24 (GP21)
- net D3_3V3: now also Data_Lines1.5 (A4)
- net D4_3V3: now reaches EEPROM_RP2040.25 (GP22)
- net D4_3V3: now also Data_Lines1.6 (A5)
- net D5_3V3: now reaches EEPROM_RP2040.26 (GP23)
- net D5_3V3: now also Data_Lines1.7 (A6)
- net D6_3V3: now reaches EEPROM_RP2040.27 (GP24)
- net D6_3V3: now also Data_Lines1.8 (A7)
- net D7_3V3: now reaches EEPROM_RP2040.28 (GP25)
- net D7_3V3: now also Data_Lines1.9 (A8)
- net UART_EE_TX: now reaches EEPROM_RP2040.32 (GP28)
- net UART_EE_TX: now also CONTROLLER_P2040.33 (GP29)
- net UART_EE_RX: now reaches EEPROM_RP2040.33 (GP29)
- net UART_EE_RX: now also CONTROLLER_P2040.32 (GP28)
- net at WIFI-ESP32C6.1 (PA02_A0_D0): now also J1.1 (Pin_1)
- net at WIFI-ESP32C6.10 (PA5_A9_D9_MISO): now also J1.8 (Pin_8)
- net at WIFI-ESP32C6.11 (PA6_A10_D10_MOSI): now also J1.9 (Pin_9)
- net at WIFI-ESP32C6.2 (PA4_A1_D1): now also J1.2 (Pin_2)
- net at WIFI-ESP32C6.3 (PA10_A2_D2): now also J1.3 (Pin_3)
- net at WIFI-ESP32C6.4 (PA11_A3_D3): now also J1.4 (Pin_4)
- net at WIFI-ESP32C6.5 (PA8_A4_D4_SDA): now also J1.5 (Pin_5)
- net at WIFI-ESP32C6.6 (PA9_A5_D5_SCL): now also J1.6 (Pin_6)
- net at WIFI-ESP32C6.7 (PB08_A6_D6_TX): now also CONTROLLER_P2040.2 (GP1)
- net at WIFI-ESP32C6.8 (PB09_A7_D7_RX): now also CONTROLLER_P2040.1 (GP0)
- net at WIFI-ESP32C6.9 (PA7_A8_D8_SCK): now also J1.7 (Pin_7)
- net D0_3V3_CO: no longer names the net of CONTROLLER_P2040.21 (GP18)
- net D0_3V3_CO: no longer Data_Lines1.1 (A1)
- net D1_3V3_CO: no longer names the net of CONTROLLER_P2040.22 (GP19)
- net D1_3V3_CO: no longer Data_Lines1.3 (A2)
- net D2_3V3_CO: no longer names the net of CONTROLLER_P2040.23 (GP20)
- net D2_3V3_CO: no longer Data_Lines1.4 (A3)
- net D3_3V3_CO: no longer names the net of CONTROLLER_P2040.24 (GP21)
- net D3_3V3_CO: no longer Data_Lines1.5 (A4)
- net D4_3V3_CO: no longer names the net of CONTROLLER_P2040.25 (GP22)
- net D4_3V3_CO: no longer Data_Lines1.6 (A5)
- net D5_3V3_CO: no longer names the net of CONTROLLER_P2040.26 (GP23)
- net D5_3V3_CO: no longer Data_Lines1.7 (A6)
- net D6_3V3_CO: no longer names the net of CONTROLLER_P2040.27 (GP24)
- net D6_3V3_CO: no longer Data_Lines1.8 (A7)
- net D7_3V3_CO: no longer names the net of CONTROLLER_P2040.28 (GP25)
- net D7_3V3_CO: no longer Data_Lines1.9 (A8)
- new net OE_Data: EEPROM_RP2040.1 (GP0)
- no-connect marks 25 -> 29

Commit message: More work on pcb
Parts:
- removed CONTROLLER_P2040, EEPROM_RP2040: WeAct-RP2040-Pico, WeAct-RP2040-Pico:WeAct-RP2040-Pico, symbol WeAct-RP2040-Pico:WeAct-RP2040-Pico
- removed J1: Conn_02x05_Pin, Connector_PinHeader_2.00mm:PinHeader_2x05_P2.00mm_Vertical, symbol Connector:Conn_01x10_Pin
- added J1: Screw_Terminal_01x03, TerminalBlock:TerminalBlock_Xinya_XY308-2.54-3P_1x03_P2.54mm_Horizontal, symbol Connector:Screw_Terminal_01x03
- added U1: rp2040-zero, kleeb-mcu:rp2040-zero-smd, symbol kleeb-mcu:rp2040-zero
- added U2: SN65176BD, SN65176BD:SOIC127P599X175-8N, symbol SN65176BD:SN65176BD
- added U3: RP2040_Stamp, RP2040_Stamp:RP2040_Stamp_SMD, symbol RP2040_Stamp:RP2040_Stamp
- WIFI-ESP32C6: footprint XIAO_PCB:MOUDLE14P-2.54-21X17.8MM -> XIAO_PCB:MOUDLE14P-SMD-2.54-21X17.8MM
Connections:
- net GND: now also J1.1 (Pin_1), U1.22 (GND), U2.5 (GND)
- net VCC_3V3: no longer WIFI-ESP32C6.12 (3V3)
- net VCC_5V: now also U1.23 (5V), U2.8 (VCC)
- new net: J1.2 (Pin_2), U2.6 (A)
- new net: J1.3 (Pin_3), U2.7 (B)
- no-connect marks 29 -> 20
Other:
- moved on the sheet: WIFI-ESP32C6

Commit message: More pcb work
Parts:
- removed U1: rp2040-zero, kleeb-mcu:rp2040-zero-smd, symbol kleeb-mcu:rp2040-zero
Changed lines of the file:
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@@
-	)
-	(symbol
-		(lib_id "kleeb-mcu:rp2040-zero")
-		(at 40.64 171.45 0)
-		(unit 1)
-		(exclude_from_sim no)
-		(in_bom yes)
-		(on_board yes)
-		(dnp no)
-		(fields_autoplaced yes)
-		(property "Reference" "U1"
-			(at 40.64 154.94 0)
-			(effects
-				(font
-					(size 1.27 1.27)
-				)
-			)
-		)
-		(property "Value" "rp2040-zero"
-			(at 40.64 157.48 0)
-			(effects
-				(font
-					(size 1.27 1.27)
-				)
-			)
-		)
-		(property "Footprint" "kleeb-mcu:rp2040-zero-smd"
-			(at 31.75 166.37 0)
-			(effects
-				(font
-					(size 1.27 1.27)
-				)
-				(hide yes)
-			)
-		)
-		(property "Datasheet" ""
-			(at 31.75 166.37 0)
-			(effects
-				(font
-					(size 1.27 1.27)
-				)
-				(hide yes)
-			)
-		)
-		(property "Description" ""
-			(at 40.64 171.45 0)
-			(effects
-				(font
-					(size 1.27 1.27)
-				)
-				(hide yes)
-			)
-		)
-		(pin "7"
-		)
-		(pin "20"
-		)
-		(pin "5"
-		)
-		(pin "12"
-		)
-		(pin "1"
-		)
-		(pin "14"
-		)
-		(pin "4"
-		)
-		(pin "21"
-		)
-		(pin "9"
-		)
-		(pin "15"
-		)
-		(pin "3"
-		)
-		(pin "10"
-		)
-		(pin "23"
-		)
-		(pin "8"
-		)
-		(pin "19"
-		)
-		(pin "18"
-		)
-		(pin "11"
-		)
-		(pin "13"
-		)
-		(pin "16"
-		)
-		(pin "17"
-		)
-		(pin "2"
-		)
-		(pin "22"
-		)
-		(pin "6"
-		)
-		(instances
-			(project "eeprom-lc_12_2"
-				(path "/bd0e159c-206b-4547-b40c-3362ba65e229"
-					(reference "U1")
-					(unit 1)
-				)
-			)
-		)
 	)
 	(symbol

Commit message: FInishing up the pcb
Parts:
- removed U3: RP2040_Stamp, RP2040_Stamp:RP2040_Stamp_SMD, symbol RP2040_Stamp:RP2040_Stamp
- added JP1: UART EE <-> ESP 1, TestPoint:TestPoint_2Pads_Pitch2.54mm_Drill0.8mm, symbol Jumper:Jumper_2_Open
- added JP2: UART EE <-> ESP 2, TestPoint:TestPoint_2Pads_Pitch2.54mm_Drill0.8mm, symbol Jumper:Jumper_2_Open
- added JP4: DMX_TX, Connector_PinHeader_1.00mm:PinHeader_1x03_P1.00mm_Horizontal, symbol Jumper:Jumper_3_Open
- added U1: Controller-RP2040, WeAct-rp2040:WeAct-RP2040-Pico, symbol WeAct-rp2040:WeAct-RP2040-Pico
- added U4: EEPROM-RP2040, WeAct-rp2040:WeAct-RP2040-Pico, symbol WeAct-rp2040:WeAct-RP2040-Pico
Connections:
- net A0_3V3: now also U4.4 (GP3)
- net A10_3V3: now also U4.16 (GP13)
- net A11_3V3: now also U4.17 (GP14)
- net A12_3V3: now also U4.18 (GP15)
- net A13_3V3: now also U4.19 (GP16)
- net A14_3V3: now also U4.20 (GP17)
- net A15_3V3: now also U4.21 (GP18)
- net A16_3V3: now also U4.22 (GP19)
- net A1_3V3: now also U4.5 (GP4)
- net A2_3V3: now also U4.7 (GP5)
- net A3_3V3: now also U4.8 (GP6)
- net A4_3V3: now also U4.9 (GP7)
- net A5_3V3: now also U4.10 (GP8)
- net A6_3V3: now also U4.11 (GP9)
- net A7_3V3: now also U4.12 (GP10)
- net A8_3V3: now also U4.13 (GP11)
- net A9_3V3: now also U4.14 (GP12)
- net D0_3V3: now also U4.25 (GP22)
- net D1_3V3: now also U4.26 (GP23)
- net D2_3V3: now also U4.27 (GP24)
- net D3_3V3: now also U4.28 (GP25)
- net D4_3V3: now also U4.30 (GP26)
- net D5_3V3: now also U4.31 (GP27)
- net D6_3V3: now also U4.32 (GP28)
- net D7_3V3: now also U4.33 (GP29)
- net GND: now also U1.38 (GND), U1.6 (GND), U4.15 (GND), U4.35 (GND), U4.38 (GND)
- net OE_3V3: now also U4.3 (GP2)
- net UART_EE_RX: now also JP1.1 (A), U1.1 (GP0), U4.1 (GP0)
- net UART_EE_TX: now also JP2.1 (A), U1.2 (GP1), U4.2 (GP1)
- net VCC_3V3: now also WIFI-ESP32C6.12 (3V3), U1.36 (3V3), U4.36 (3V3)
- net VCC_5V: now also U2.2 (~{RE}), U2.3 (DE), U1.40 (VBUS), U4.40 (VBUS)
- net UART_ESP_TX: now reaches WIFI-ESP32C6.7 (PB08_A6_D6_TX)
- net UART_ESP_TX: now also JP1.2 (B), U1.24 (GP21)
- net UART_ESP_RX: now reaches WIFI-ESP32C6.8 (PB09_A7_D7_RX)
- net UART_ESP_RX: now also JP2.2 (B), U1.23 (GP20)
- net DMX_TX: now reaches U2.4 (D)
- net DMX_TX: now also JP4.2 (C)
- new net DMX_TX_CON: JP4.3 (B), U1.28 (GP25)
- new net DMX_TX_EE: JP4.1 (A), U4.23 (GP20)
- no-connect marks 20 -> 70
Other:
- moved on the sheet: Address_0_7, Address_16_OE1, Address_8_15, Data_Lines1, WIFI-ESP32C6

Commit message: Fix wrong pinheaders
Parts:
- J1: footprint TerminalBlock:TerminalBlock_Xinya_XY308-2.54-3P_1x03_P2.54mm_Horizontal -> Connector_PinHeader_2.54mm:PinHeader_1x03_P2.54mm_Vertical
- JP4: footprint Connector_PinHeader_1.00mm:PinHeader_1x03_P1.00mm_Horizontal -> Connector_PinHeader_2.54mm:PinHeader_1x03_P2.54mm_Horizontal
Changed lines of the file:
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@@
 			)
 		)
-		(property "Footprint" "Connector_PinHeader_1.00mm:PinHeader_1x03_P1.00mm_Horizontal"
+		(property "Footprint" "Connector_PinHeader_2.54mm:PinHeader_1x03_P2.54mm_Horizontal"
 			(at 161.29 115.57 0)
 			(effects
@@
 			)
 		)
-		(property "Footprint" "TerminalBlock:TerminalBlock_Xinya_XY308-2.54-3P_1x03_P2.54mm_Horizontal"
+		(property "Footprint" "Connector_PinHeader_2.54mm:PinHeader_1x03_P2.54mm_Vertical"
 			(at 146.05 177.8 0)
 			(effects

Commit message: Finished up the eeprom pcb
Parts:
- added C1, C2, C3, C4, C5, C6, C7, C8: C_Small, Capacitor_SMD:C_0603_1608Metric_Pad1.08x0.95mm_HandSolder, symbol Device:C_Small
Connections:
- net GND: now also C1.1, C2.1, C3.1, C4.1, C5.1, C6.1, C7.1, C8.1
- net VCC_5V: now also C1.2, C2.2, C3.2, C4.2, C5.2, C6.2, C7.2, C8.2
- removed net VCC_3V3: Address_0_7.10 (OE), Address_0_7.2 (VCCA), Address_16_OE1.10 (OE), Address_16_OE1.2 (VCCA), Address_8_15.10 (OE), Address_8_15.2 (VCCA), Data_Lines1.10 (OE), Data_Lines1.2 (VCCA), U1.36 (3V3), U4.36 (3V3), WIFI-ESP32C6.12 (3V3)
- new net VCC_3V3_CON: Address_16_OE1.10 (OE), Address_16_OE1.2 (VCCA), U1.36 (3V3)
- new net VCC_3V3_EE: Address_0_7.10 (OE), Address_0_7.2 (VCCA), Data_Lines1.10 (OE), Data_Lines1.2 (VCCA), U4.36 (3V3)
- new net VCC_3V3_ESP: Address_8_15.10 (OE), Address_8_15.2 (VCCA), WIFI-ESP32C6.12 (3V3)
