File: eeprom-lc_12_2/eeprom-lc_12_2.kicad_pcb (KiCad board)
At the start: 2 copper layers, 9 parts, among them U5 TXS0108EPW, U6 TXS0108EPW

Commit message: Some work on eeprom code and pcb
Parts:
- added J1: Conn_02x05_Pin, Connector_PinHeader_2.00mm:PinHeader_2x05_P2.00mm_Vertical, F.Cu at (90.9, 55.9)
- CONTROLLER_P2040, EEPROM_RP2040: footprint WeAct-rp2040:WeAct-RP2040-Pico -> WeAct-RP2040-Pico:WeAct-RP2040-Pico
- WIFI-ESP32C6: value MOUDLE-SEEEDUINO-XIAO -> WeAct-RP2040-Pico; footprint XIAO-rp2040:MOUDLE14P-2.54-21X17.8MM -> XIAO_PCB:MOUDLE14P-2.54-21X17.8MM
- moved WIFI-ESP32C6 105.5 mm to (86.4, 71.1), turned to -90 degrees
- moved EEPROM_RP2040 94.0 mm to (146.0, 87.5), turned to -90 degrees
- moved Address_16_OE1 75.6 mm to (88.9, 88.9), turned to -90 degrees
- moved CONTROLLER_P2040 66.0 mm to (146.0, 62.1), turned to -90 degrees
- moved Address_8_15 52.6 mm to (121.9, 61.0), turned to 180 degrees
- moved EEPROM_SLOT1 42.9 mm to (99.1, 55.9), turned to 180 degrees
- moved Address_0_7 37.2 mm to (137.2, 60.6)
- moved Data_Controller1 18.1 mm to (154.9, 63.5), turned to 90 degrees
- moved Data_EEPROM1 10.0 mm to (145.0, 88.6), turned to 90 degrees
- renumbered U5 to Data_Controller1, U6 to Data_EEPROM1
Connections:
- Address_0_7 pad 1: unconnected-(Address_0_7-A1-Pad1) -> /A0_3V3
- Address_0_7 pad 10: unconnected-(Address_0_7-OE-Pad10) -> /VCC_3V3
- Address_0_7 pad 3: unconnected-(Address_0_7-A2-Pad3) -> /A1_3V3
- Address_0_7 pad 4: unconnected-(Address_0_7-A3-Pad4) -> /A2_3V3
- Address_0_7 pad 5: unconnected-(Address_0_7-A4-Pad5) -> /A3_3V3
- Address_0_7 pad 6: unconnected-(Address_0_7-A5-Pad6) -> /A4_3V3
- Address_0_7 pad 7: unconnected-(Address_0_7-A6-Pad7) -> /A5_3V3
- Address_0_7 pad 8: unconnected-(Address_0_7-A7-Pad8) -> /A6_3V3
- Address_0_7 pad 9: unconnected-(Address_0_7-A8-Pad9) -> /A7_3V3
- Address_16_OE1 pad 1: unconnected-(Address_16_OE1-A1-Pad1) -> /A16_3V3
- Address_16_OE1 pad 10: unconnected-(Address_16_OE1-OE-Pad10) -> /VCC_3V3
- Address_16_OE1 pad 3: unconnected-(Address_16_OE1-A2-Pad3) -> /OE_3V3
- Address_8_15 pad 1: unconnected-(Address_8_15-A1-Pad1) -> /A8_3V3
- Address_8_15 pad 10: unconnected-(Address_8_15-OE-Pad10) -> /VCC_3V3
- Address_8_15 pad 3: unconnected-(Address_8_15-A2-Pad3) -> /A9_3V3
- Address_8_15 pad 4: unconnected-(Address_8_15-A3-Pad4) -> /A10_3V3
- Address_8_15 pad 5: unconnected-(Address_8_15-A4-Pad5) -> /A11_3V3
- Address_8_15 pad 6: unconnected-(Address_8_15-A5-Pad6) -> /A12_3V3
- Address_8_15 pad 7: unconnected-(Address_8_15-A6-Pad7) -> /A13_3V3
- Address_8_15 pad 8: unconnected-(Address_8_15-A7-Pad8) -> /A14_3V3
- Address_8_15 pad 9: unconnected-(Address_8_15-A8-Pad9) -> /A15_3V3
- CONTROLLER_P2040 pad 1: unconnected-(CONTROLLER_P2040-GP0-Pad1) -> Net-(CONTROLLER_P2040-GP0)
- CONTROLLER_P2040 pad 10: unconnected-(CONTROLLER_P2040-GP8-Pad10) -> /A5_3V3
- CONTROLLER_P2040 pad 11: unconnected-(CONTROLLER_P2040-GP9-Pad11) -> /A6_3V3
- CONTROLLER_P2040 pad 12: unconnected-(CONTROLLER_P2040-GP10-Pad12) -> /A7_3V3
- CONTROLLER_P2040 pad 13: unconnected-(CONTROLLER_P2040-GP11-Pad13) -> /A8_3V3
- CONTROLLER_P2040 pad 14: unconnected-(CONTROLLER_P2040-GP12-Pad14) -> /A9_3V3
- CONTROLLER_P2040 pad 16: unconnected-(CONTROLLER_P2040-GP13-Pad16) -> /A10_3V3
- CONTROLLER_P2040 pad 17: unconnected-(CONTROLLER_P2040-GP14-Pad17) -> /A11_3V3
- CONTROLLER_P2040 pad 18: unconnected-(CONTROLLER_P2040-GP15-Pad18) -> /A12_3V3
- CONTROLLER_P2040 pad 19: unconnected-(CONTROLLER_P2040-GP16-Pad19) -> /A13_3V3
- CONTROLLER_P2040 pad 2: unconnected-(CONTROLLER_P2040-GP1-Pad2) -> Net-(CONTROLLER_P2040-GP1)
- CONTROLLER_P2040 pad 20: unconnected-(CONTROLLER_P2040-GP17-Pad20) -> /A14_3V3
- CONTROLLER_P2040 pad 21: unconnected-(CONTROLLER_P2040-GP18-Pad21) -> /A16_3V3
- CONTROLLER_P2040 pad 22: unconnected-(CONTROLLER_P2040-GP19-Pad22) -> /A15_3V3
- CONTROLLER_P2040 pad 23: unconnected-(CONTROLLER_P2040-GP20-Pad23) -> Net-(CONTROLLER_P2040-GP20)
- CONTROLLER_P2040 pad 24: unconnected-(CONTROLLER_P2040-GP21-Pad24) -> Net-(CONTROLLER_P2040-GP21)
- CONTROLLER_P2040 pad 25: unconnected-(CONTROLLER_P2040-GP22-Pad25) -> /D0_3V3_CO
- CONTROLLER_P2040 pad 26: unconnected-(CONTROLLER_P2040-GP23-Pad26) -> /D1_3V3_CO
- CONTROLLER_P2040 pad 27: unconnected-(CONTROLLER_P2040-GP24-Pad27) -> /D2_3V3_CO
- CONTROLLER_P2040 pad 28: unconnected-(CONTROLLER_P2040-GP25-Pad28) -> /D3_3V3_CO
- CONTROLLER_P2040 pad 3: unconnected-(CONTROLLER_P2040-GP2-Pad3) -> /OE_3V3
- CONTROLLER_P2040 pad 30: unconnected-(CONTROLLER_P2040-GP26-Pad30) -> /D4_3V3_CO
- CONTROLLER_P2040 pad 31: unconnected-(CONTROLLER_P2040-GP27-Pad31) -> /D5_3V3_CO
- CONTROLLER_P2040 pad 32: unconnected-(CONTROLLER_P2040-GP28-Pad32) -> /D6_3V3_CO
- CONTROLLER_P2040 pad 33: unconnected-(CONTROLLER_P2040-GP29-Pad33) -> /D7_3V3_CO
- CONTROLLER_P2040 pad 36: unconnected-(CONTROLLER_P2040-3V3-Pad36) -> /VCC_3V3
- CONTROLLER_P2040 pad 38: unconnected-(CONTROLLER_P2040-GND-Pad38) -> /GND
- CONTROLLER_P2040 pad 39: unconnected-(CONTROLLER_P2040-VIN-Pad39) -> /VCC_5V
- CONTROLLER_P2040 pad 4: unconnected-(CONTROLLER_P2040-GP3-Pad4) -> /A0_3V3
- CONTROLLER_P2040 pad 5: unconnected-(CONTROLLER_P2040-GP4-Pad5) -> /A1_3V3
- CONTROLLER_P2040 pad 7: unconnected-(CONTROLLER_P2040-GP5-Pad7) -> /A2_3V3
- CONTROLLER_P2040 pad 8: unconnected-(CONTROLLER_P2040-GP6-Pad8) -> /A3_3V3
- CONTROLLER_P2040 pad 9: unconnected-(CONTROLLER_P2040-GP7-Pad9) -> /A4_3V3
- Data_Controller1 pad 1: unconnected-(U5-A1-Pad1) -> /D0_3V3_CO
- Data_Controller1 pad 10: unconnected-(U5-OE-Pad10) -> /VCC_3V3
- Data_Controller1 pad 3: unconnected-(U5-A2-Pad3) -> /D1_3V3_CO
- Data_Controller1 pad 4: unconnected-(U5-A3-Pad4) -> /D2_3V3_CO
- Data_Controller1 pad 5: unconnected-(U5-A4-Pad5) -> /D3_3V3_CO
- Data_Controller1 pad 6: unconnected-(U5-A5-Pad6) -> /D4_3V3_CO
- Data_Controller1 pad 7: unconnected-(U5-A6-Pad7) -> /D5_3V3_CO
- Data_Controller1 pad 8: unconnected-(U5-A7-Pad8) -> /D6_3V3_CO
- Data_Controller1 pad 9: unconnected-(U5-A8-Pad9) -> /D7_3V3_CO
- Data_EEPROM1 pad 1: unconnected-(U6-A1-Pad1) -> /D0_3V3_EE
- Data_EEPROM1 pad 10: unconnected-(U6-OE-Pad10) -> /OE_Data
- Data_EEPROM1 pad 3: unconnected-(U6-A2-Pad3) -> /D1_3V3_EE
- Data_EEPROM1 pad 4: unconnected-(U6-A3-Pad4) -> /D2_3V3_EE
- Data_EEPROM1 pad 5: unconnected-(U6-A4-Pad5) -> /D3_3V3_EE
- Data_EEPROM1 pad 6: unconnected-(U6-A5-Pad6) -> /D4_3V3_EE
- Data_EEPROM1 pad 7: unconnected-(U6-A6-Pad7) -> /D5_3V3_EE
- Data_EEPROM1 pad 8: unconnected-(U6-A7-Pad8) -> /D6_3V3_EE
- Data_EEPROM1 pad 9: unconnected-(U6-A8-Pad9) -> /D7_3V3_EE
- EEPROM_RP2040 pad 1: unconnected-(EEPROM_RP2040-GP0-Pad1) -> /OE_Data
- EEPROM_RP2040 pad 10: unconnected-(EEPROM_RP2040-GP8-Pad10) -> /A5_3V3
- EEPROM_RP2040 pad 11: unconnected-(EEPROM_RP2040-GP9-Pad11) -> /A6_3V3
- EEPROM_RP2040 pad 12: unconnected-(EEPROM_RP2040-GP10-Pad12) -> /A7_3V3
- EEPROM_RP2040 pad 13: unconnected-(EEPROM_RP2040-GP11-Pad13) -> /A8_3V3
- EEPROM_RP2040 pad 14: unconnected-(EEPROM_RP2040-GP12-Pad14) -> /A9_3V3
- EEPROM_RP2040 pad 16: unconnected-(EEPROM_RP2040-GP13-Pad16) -> /A10_3V3
- EEPROM_RP2040 pad 17: unconnected-(EEPROM_RP2040-GP14-Pad17) -> /A11_3V3
- EEPROM_RP2040 pad 18: unconnected-(EEPROM_RP2040-GP15-Pad18) -> /A12_3V3
- EEPROM_RP2040 pad 19: unconnected-(EEPROM_RP2040-GP16-Pad19) -> /A13_3V3
- EEPROM_RP2040 pad 20: unconnected-(EEPROM_RP2040-GP17-Pad20) -> /A14_3V3
- EEPROM_RP2040 pad 21: unconnected-(EEPROM_RP2040-GP18-Pad21) -> /A16_3V3
- EEPROM_RP2040 pad 22: unconnected-(EEPROM_RP2040-GP19-Pad22) -> /A15_3V3
- EEPROM_RP2040 pad 23: unconnected-(EEPROM_RP2040-GP20-Pad23) -> Net-(CONTROLLER_P2040-GP21)
- EEPROM_RP2040 pad 24: unconnected-(EEPROM_RP2040-GP21-Pad24) -> Net-(CONTROLLER_P2040-GP20)
- EEPROM_RP2040 pad 25: unconnected-(EEPROM_RP2040-GP22-Pad25) -> /D0_3V3_EE
- EEPROM_RP2040 pad 26: unconnected-(EEPROM_RP2040-GP23-Pad26) -> /D1_3V3_EE
- EEPROM_RP2040 pad 27: unconnected-(EEPROM_RP2040-GP24-Pad27) -> /D2_3V3_EE
- EEPROM_RP2040 pad 28: unconnected-(EEPROM_RP2040-GP25-Pad28) -> /D3_3V3_EE
- EEPROM_RP2040 pad 3: unconnected-(EEPROM_RP2040-GP2-Pad3) -> /OE_3V3
- EEPROM_RP2040 pad 30: unconnected-(EEPROM_RP2040-GP26-Pad30) -> /D4_3V3_EE
- EEPROM_RP2040 pad 31: unconnected-(EEPROM_RP2040-GP27-Pad31) -> /D5_3V3_EE
- EEPROM_RP2040 pad 32: unconnected-(EEPROM_RP2040-GP28-Pad32) -> /D6_3V3_EE
- EEPROM_RP2040 pad 33: unconnected-(EEPROM_RP2040-GP29-Pad33) -> /D7_3V3_EE
- EEPROM_RP2040 pad 36: unconnected-(EEPROM_RP2040-3V3-Pad36) -> /VCC_3V3
- EEPROM_RP2040 pad 38: unconnected-(EEPROM_RP2040-GND-Pad38) -> /GND
- EEPROM_RP2040 pad 39: unconnected-(EEPROM_RP2040-VIN-Pad39) -> /VCC_5V
- EEPROM_RP2040 pad 4: unconnected-(EEPROM_RP2040-GP3-Pad4) -> /A0_3V3
- EEPROM_RP2040 pad 5: unconnected-(EEPROM_RP2040-GP4-Pad5) -> /A1_3V3
- EEPROM_RP2040 pad 7: unconnected-(EEPROM_RP2040-GP5-Pad7) -> /A2_3V3
- EEPROM_RP2040 pad 8: unconnected-(EEPROM_RP2040-GP6-Pad8) -> /A3_3V3
- EEPROM_RP2040 pad 9: unconnected-(EEPROM_RP2040-GP7-Pad9) -> /A4_3V3
- EEPROM_SLOT1 pad 1: /VCC_5V -> unconnected-(EEPROM_SLOT1-VPP-Pad1)
- EEPROM_SLOT1 pad 24: /GND -> unconnected-(EEPROM_SLOT1-~G-Pad24)
- EEPROM_SLOT1 pad 31: /VCC_5V -> unconnected-(EEPROM_SLOT1-~P-Pad31)
- WIFI-ESP32C6 pad 1: unconnected-(WIFI-ESP32C6-PA02_A0_D0-Pad1) -> Net-(J1-Pin_1)
- WIFI-ESP32C6 pad 10: unconnected-(WIFI-ESP32C6-PA5_A9_D9_MISO-Pad10) -> Net-(J1-Pin_8)
- WIFI-ESP32C6 pad 11: unconnected-(WIFI-ESP32C6-PA6_A10_D10_MOSI-Pad11) -> Net-(J1-Pin_9)
- WIFI-ESP32C6 pad 12: unconnected-(WIFI-ESP32C6-3V3-Pad12) -> /VCC_3V3
- WIFI-ESP32C6 pad 2: unconnected-(WIFI-ESP32C6-PA4_A1_D1-Pad2) -> Net-(J1-Pin_2)
- WIFI-ESP32C6 pad 3: unconnected-(WIFI-ESP32C6-PA10_A2_D2-Pad3) -> Net-(J1-Pin_3)
- WIFI-ESP32C6 pad 4: unconnected-(WIFI-ESP32C6-PA11_A3_D3-Pad4) -> Net-(J1-Pin_4)
- WIFI-ESP32C6 pad 5: unconnected-(WIFI-ESP32C6-PA8_A4_D4_SDA-Pad5) -> Net-(J1-Pin_5)
- WIFI-ESP32C6 pad 6: unconnected-(WIFI-ESP32C6-PA9_A5_D5_SCL-Pad6) -> Net-(J1-Pin_6)
- WIFI-ESP32C6 pad 7: unconnected-(WIFI-ESP32C6-PB08_A6_D6_TX-Pad7) -> Net-(CONTROLLER_P2040-GP1)
- WIFI-ESP32C6 pad 8: unconnected-(WIFI-ESP32C6-PB09_A7_D7_RX-Pad8) -> Net-(CONTROLLER_P2040-GP0)
- WIFI-ESP32C6 pad 9: unconnected-(WIFI-ESP32C6-PA7_A8_D8_SCK-Pad9) -> Net-(J1-Pin_7)
Routing:
- net /VCC_5V: track 0.00 -> 252.7 mm, vias 0 -> 10
- net /GND: track 0.00 -> 216.7 mm, vias 0 -> 5
- net Net-(CONTROLLER_P2040-GP0): track 0.00 -> 102.9 mm
- net /VCC_3V3: track 0.00 -> 101.4 mm, vias 0 -> 2
- net /D0_5V: track 0.00 -> 90.0 mm, vias 0 -> 2
- net /D1_5V: track 0.00 -> 84.3 mm
- net /D2_5V: track 0.00 -> 84.2 mm
- net Net-(CONTROLLER_P2040-GP1): track 0.00 -> 83.3 mm
- net /D3_5V: track 0.00 -> 66.2 mm
- net /D4_5V: track 0.00 -> 64.9 mm
- net /D5_5V: track 0.00 -> 63.6 mm
- net /A16_3V3: track 0.00 -> 62.8 mm, vias 0 -> 1
- net /D6_5V: track 0.00 -> 62.4 mm
- net /D7_5V: track 0.00 -> 61.6 mm
- net /A0_3V3: track 0.00 -> 53.1 mm
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Other:
- board outline added: 97 x 48.3 mm

Commit message: More work on pcb
Parts:
- removed CONTROLLER_P2040, EEPROM_RP2040: WeAct-RP2040-Pico, WeAct-RP2040-Pico:WeAct-RP2040-Pico
- removed Data_EEPROM1: TXS0108EPW, Package_SO:TSSOP-20_4.4x6.5mm_P0.65mm
- added U1: rp2040-zero, kleeb-mcu:rp2040-zero-smd, F.Cu at (132.1, 88.9)
- added U2: SN65176BD, SN65176BD:SOIC127P599X175-8N, F.Cu at (160.0, 91.4)
- added U3: RP2040_Stamp, RP2040_Stamp:RP2040_Stamp_SMD, F.Cu at (160.0, 63.9)
- J1: value Conn_02x05_Pin -> Screw_Terminal_01x03; footprint Connector_PinHeader_2.00mm:PinHeader_2x05_P2.00mm_Vertical -> TerminalBlock:TerminalBlock_Xinya_XY308-2.54-3P_1x03_P2.54mm_Horizontal
- WIFI-ESP32C6: footprint XIAO_PCB:MOUDLE14P-2.54-21X17.8MM -> XIAO_PCB:MOUDLE14P-SMD-2.54-21X17.8MM
- moved J1 85.9 mm to (170.2, 88.9)
- moved Data_Lines1 48.3 mm to (106.7, 61.0), turned to -90 degrees
- moved Address_8_15 25.4 mm to (106.7, 81.3), turned to -90 degrees
- moved Address_0_7 15.2 mm to (124.5, 68.9), turned to 90 degrees
- moved WIFI-ESP32C6 10.4 mm to (77.4, 76.4), turned to 0 degrees
- moved Address_16_OE1 5.08 mm to (83.8, 88.9), turned to 90 degrees
- renumbered Data_Controller1 to Data_Lines1
Connections:
- Data_Lines1 pad 1: /D0_3V3_CO -> /D0_3V3
- Data_Lines1 pad 3: /D1_3V3_CO -> /D1_3V3
- Data_Lines1 pad 4: /D2_3V3_CO -> /D2_3V3
- Data_Lines1 pad 5: /D3_3V3_CO -> /D3_3V3
- Data_Lines1 pad 6: /D4_3V3_CO -> /D4_3V3
- Data_Lines1 pad 7: /D5_3V3_CO -> /D5_3V3
- Data_Lines1 pad 8: /D6_3V3_CO -> /D6_3V3
- Data_Lines1 pad 9: /D7_3V3_CO -> /D7_3V3
- J1 pad 1: Net-(J1-Pin_1) -> /GND
- WIFI-ESP32C6 pad 1: Net-(J1-Pin_1) -> unconnected-(WIFI-ESP32C6-PA02_A0_D0-Pad1)
- WIFI-ESP32C6 pad 10: Net-(J1-Pin_8) -> unconnected-(WIFI-ESP32C6-PA5_A9_D9_MISO-Pad10)
- WIFI-ESP32C6 pad 11: Net-(J1-Pin_9) -> unconnected-(WIFI-ESP32C6-PA6_A10_D10_MOSI-Pad11)
- WIFI-ESP32C6 pad 12: /VCC_3V3 -> unconnected-(WIFI-ESP32C6-3V3-Pad12)
- WIFI-ESP32C6 pad 2: Net-(J1-Pin_2) -> unconnected-(WIFI-ESP32C6-PA4_A1_D1-Pad2)
- WIFI-ESP32C6 pad 3: Net-(J1-Pin_3) -> unconnected-(WIFI-ESP32C6-PA10_A2_D2-Pad3)
- WIFI-ESP32C6 pad 4: Net-(J1-Pin_4) -> unconnected-(WIFI-ESP32C6-PA11_A3_D3-Pad4)
- WIFI-ESP32C6 pad 5: Net-(J1-Pin_5) -> unconnected-(WIFI-ESP32C6-PA8_A4_D4_SDA-Pad5)
- WIFI-ESP32C6 pad 6: Net-(J1-Pin_6) -> unconnected-(WIFI-ESP32C6-PA9_A5_D5_SCL-Pad6)
- WIFI-ESP32C6 pad 7: Net-(CONTROLLER_P2040-GP1) -> unconnected-(WIFI-ESP32C6-PB08_A6_D6_TX-Pad7)
- WIFI-ESP32C6 pad 8: Net-(CONTROLLER_P2040-GP0) -> unconnected-(WIFI-ESP32C6-PB09_A7_D7_RX-Pad8)
- WIFI-ESP32C6 pad 9: Net-(J1-Pin_7) -> unconnected-(WIFI-ESP32C6-PA7_A8_D8_SCK-Pad9)
Routing:
- net /VCC_5V: track 252.7 -> 21.2 mm, vias 10 -> 0
- net Net-(CONTROLLER_P2040-GP0): track 102.9 -> 0.00 mm
- net /VCC_3V3: track 101.4 -> 0.00 mm, vias 2 -> 0
- net /GND: track 216.7 -> 129.3 mm, vias 5 -> 0
- net /D0_5V: track 90.0 -> 4.83 mm, vias 2 -> 0
- net Net-(CONTROLLER_P2040-GP1): track 83.3 -> 0.00 mm
- net /D1_5V: track 84.3 -> 7.61 mm
- net /D2_5V: track 84.2 -> 9.64 mm
- net /D3_5V: track 66.2 -> 0.00 mm
- net /A16_3V3: track 62.8 -> 0.00 mm, vias 1 -> 0
- net /D7_5V: track 61.6 -> 0.00 mm
- net /D5_5V: track 63.6 -> 8.30 mm
- net /D6_5V: track 62.4 -> 7.25 mm
- net /D4_5V: track 64.9 -> 10.0 mm
- net /A0_3V3: track 53.1 -> 0.00 mm
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
Commit message: More pcb work
Parts:
- moved J1 5.08 mm to (170.2, 94.0), turned to 90 degrees
Routing:
- net Net-(J1-Pin_3): track 0.00 -> 8.48 mm
- net /GND: track 129.3 -> 137.3 mm
- net Net-(J1-Pin_2): track 0.00 -> 7.95 mm
Changed lines of the file:
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@@
 	(footprint "TerminalBlock:TerminalBlock_Xinya_XY308-2.54-3P_1x03_P2.54mm_Horizontal"
 		(layer "F.Cu")
-		(at 170.18 88.9 -90)
+		(at 170.18 93.98 90)
 		(descr "Terminal Block Xinya XY308-2.54-3P, 3 pins, pitch 2.54mm, size 8.12x6.5mm^2, drill diameter 1.2mm, pad diameter 2mm, see http://www.xinyaelectronic.com/product/xy308-254, script-generated using https://gitlab.com/kicad/libraries/kicad-footprint-generator/-/tree/master/scripts/TerminalBlock_Xinya")
 		(tags "THT Terminal Block Xinya XY308-2.54-3P pitch 2.54mm size 8.12x6.5mm^2 drill 1.2mm pad 2mm")
 		(property "Reference" "J1"
-			(at 2.54 -4.22 90)
+			(at 2.54 -4.22 270)
 			(layer "F.SilkS")
 			(effects
@@
 		)
 		(property "Value" "Screw_Terminal_01x03"
-			(at 2.54 4.52 90)
+			(at 2.54 4.52 270)
 			(layer "F.Fab")
 			(effects
@@
 		)
 		(property "Footprint" "TerminalBlock:TerminalBlock_Xinya_XY308-2.54-3P_1x03_P2.54mm_Horizontal"
-			(at 0 0 -90)
+			(at 0 0 90)
 			(unlocked yes)
 			(layer "F.Fab")
@@
 		)
 		(property "Datasheet" ""
-			(at 0 0 -90)
+			(at 0 0 90)
 			(unlocked yes)
 			(layer "F.Fab")
@@
 		)
 		(property "Description" "Generic screw terminal, single row, 01x03, script generated (kicad-library-utils/schlib/autogen/connector/)"
-			(at 0 0 -90)
+			(at 0 0 90)
 			(unlocked yes)
 			(layer "F.Fab")
@@
 		(attr through_hole)
 		(fp_line
-			(start -1.88 3.76)
-			(end -1.08 3.76)
+			(start 6.721 -3.22)
+			(end 6.721 3.52)
 			(stroke
 				(width 0.12)
@@
 		)
 		(fp_line
-			(start -1.64 3.52)
-			(end 6.721 3.52)
+			(start -1.64 -3.22)
+			(end 6.721 -3.22)
 			(stroke
 				(width 0.12)
@@
 		)
 		(fp_line
-			(start -1.88 2.72)
-			(end -1.88 3.76)
+			(start -1.64 -3.22)
+			(end -1.64 3.52)
 			(stroke
 				(width 0.12)
@@
 		)
 		(fp_line
-			(start -1.64 2.6)
-			(end 6.721 2.6)
+			(start -1.64 -1.501)
+			(end 6.721 -1.501)
 			(stroke
 				(width 0.12)
@@
 		)
 		(fp_line
-			(start -1.64 -1.501)
-			(end 6.721 -1.501)
+			(start -1.64 2.6)
+			(end 6.721 2.6)
 			(stroke
 				(width 0.12)
@@
 		)
 		(fp_line
-			(start -1.64 -3.22)
-			(end -1.64 3.52)
+			(start -1.88 2.72)
+			(end -1.88 3.76)
 			(stroke
 				(width 0.12)
@@
 		)
 		(fp_line
-			(start -1.64 -3.22)
-			(end 6.721 -3.22)
+			(start -1.64 3.52)
+			(end 6.721 3.52)
 			(stroke
 				(width 0.12)
@@
 		)
 		(fp_line
-			(start 6.721 -3.22)
-			(end 6.721 3.52)
+			(start -1.88 3.76)
+			(end -1.08 3.76)
 			(stroke
 				(width 0.12)
@@
 		)
 		(fp_line
-			(start -2.02 3.9)
-			(end 7.11 3.9)
+			(start 7.11 -3.6)
+			(end -2.02 -3.6)
 			(stroke
 				(width 0.05)
@@
 		)
 		(fp_line
-			(start 7.11 3.9)
-			(end 7.11 -3.6)
+			(start -2.02 -3.6)
+			(end -2.02 3.9)
 			(stroke
 				(width 0.05)
@@
 		)
 		(fp_line
-			(start -2.02 -3.6)
-			(end -2.02 3.9)
+			(start 7.11 3.9)
+			(end 7.11 -3.6)
 			(stroke
 				(width 0.05)
@@
 		)
 		(fp_line
-			(start 7.11 -3.6)
-			(end -2.02 -3.6)
+			(start -2.02 3.9)
+			(end 7.11 3.9)
 			(stroke
 				(width 0.05)
@@
 		)
 		(fp_line
-			(start -0.72 3.4)
-			(end -1.52 2.6)
+			(start 6.6 -3.1)
+			(end 6.6 3.4)
 			(stroke
 				(width 0.1)
@@
 		)
 		(fp_line
-			(start 6.6 3.4)
-			(end -0.72 3.4)
+			(start -1.52 -3.1)
+			(end 6.6 -3.1)
 			(stroke
 				(width 0.1)
@@
 		)
 		(fp_line
-			(start -1.52 2.6)
-			(end 6.6 2.6)
+			(start -1.52 -1.5)
+			(end 6.6 -1.5)
 			(stroke
 				(width 0.1)
@@
 		)
 		(fp_line
-			(start -1.52 2.6)
-			(end -1.52 -3.1)
+			(start 5.717 -0.759)
+			(end 4.322 0.637)
 			(stroke
 				(width 0.1)
@@
 		)
 		(fp_line
-			(start -1.52 1.6)
-			(end 6.6 1.6)
+			(start 3.177 -0.759)
+			(end 1.782 0.637)
 			(stroke
 				(width 0.1)
@@
 		)
 		(fp_line
-			(start 0.759 -0.637)
-			(end -0.637 0.759)
+			(start 0.637 -0.759)
+			(end -0.759 0.637)
 			(stroke
 				(width 0.1)
@@
 		)
 		(fp_line
-			(start 3.299 -0.637)
-			(end 1.904 0.759)
+			(start 5.839 -0.637)
+			(end 4.444 0.759)
 			(stroke
 				(width 0.1)
@@
 		)
 		(fp_line
-			(start 5.839 -0.637)
-			(end 4.444 0.759)
+			(start 3.299 -0.637)
+			(end 1.904 0.759)
 			(stroke
 				(width 0.1)
@@
 		)
 		(fp_line
-			(start 0.637 -0.759)
-			(end -0.759 0.637)
+			(start 0.759 -0.637)
+			(end -0.637 0.759)
 			(stroke
 				(width 0.1)
@@
 		)
 		(fp_line
-			(start 3.177 -0.759)
-			(end 1.782 0.637)
+			(start -1.52 1.6)
+			(end 6.6 1.6)
 			(stroke
 				(width 0.1)
@@
 		)
 		(fp_line
-			(start 5.717 -0.759)
-			(end 4.322 0.637)
+			(start -1.52 2.6)
+			(end -1.52 -3.1)
 			(stroke
 				(width 0.1)
@@
 		)
 		(fp_line
-			(start -1.52 -1.5)
-			(end 6.6 -1.5)
+			(start -1.52 2.6)
+			(end 6.6 2.6)
 			(stroke
 				(width 0.1)
@@
 		)
 		(fp_line
-			(start -1.52 -3.1)
-			(end 6.6 -3.1)
+			(start 6.6 3.4)
+			(end -0.72 3.4)
 			(stroke
 				(width 0.1)
@@
 		)
 		(fp_line
-			(start 6.6 -3.1)
-			(end 6.6 3.4)
+			(start -0.72 3.4)
+			(end -1.52 2.6)
 			(stroke
 				(width 0.1)
@@
 		)
 		(fp_circle
-			(center 0 0)
-			(end 1 0)
+			(center 5.08 0)
+			(end 6.08 0)
 			(stroke
 				(width 0.1)
@@
 		)
 		(fp_circle
-			(center 5.08 0)
-			(end 6.08 0)
+			(center 0 0)
+			(end 1 0)
 			(stroke
 				(width 0.1)
@@
 		)
 		(fp_text user "${REFERENCE}"
-			(at 2.54 2.15 90)
+			(at 2.54 2.15 270)
 			(layer "F.Fab")
 			(effects
@@
 		)
 		(pad "1" thru_hole rect
-			(at 0 0 270)
+			(at 0 0 90)
 			(size 2 2)
 			(drill 1.2)
@@
 		)
 		(pad "2" thru_hole circle
-			(at 2.54 0 270)
+			(at 2.54 0 90)
 			(size 2 2)
 			(drill 1.2)
@@
 		)
 		(pad "3" thru_hole circle
-			(at 5.08 0 270)
+			(at 5.08 0 90)
 			(size 2 2)
 			(drill 1.2)
@@
 	)
 	(segment
+		(start 162.49 93.345)
+		(end 169.545 93.345)
+		(width 0.3)
+		(layer "F.Cu")
+		(net 18)
+	)
+	(segment
 		(start 99.06 55.88)
 		(end 100.844248 57.664248)
@@
 	)
 	(segment
+		(start 169.545 93.345)
+		(end 170.18 93.98)
+		(width 0.3)
+		(layer "F.Cu")
+		(net 18)
+	)
+	(segment
 		(start 100.844248 57.664248)
 		(end 100.844248 59.40946)
@@
 		(net 95)
 	)
+	(segment
+		(start 162.49 92.075)
+		(end 169.545 92.075)
+		(width 0.3)
+		(layer "F.Cu")
+		(net 105)
+	)
+	(segment
+		(start 169.545 92.075)
+		(end 170.18 91.44)
+		(width 0.3)
+		(layer "F.Cu")
+		(net 105)
+	)
+	(segment
+		(start 162.49 90.805)
+		(end 168.275 90.805)
+		(width 0.3)
+		(layer "F.Cu")
+		(net 106)
+	)
+	(segment
+		(start 168.275 90.805)
+		(end 170.18 88.9)
+		(width 0.3)
+		(layer "F.Cu")
+		(net 106)
+	)
 )

Commit message: FInishing up the pcb
Parts:
- removed U3: RP2040_Stamp, RP2040_Stamp:RP2040_Stamp_SMD
- added JP1: UART EE <-> ESP 1, TestPoint:TestPoint_2Pads_Pitch2.54mm_Drill0.8mm, F.Cu at (86.0, 87.8)
- added JP2: UART EE <-> ESP 2, TestPoint:TestPoint_2Pads_Pitch2.54mm_Drill0.8mm, F.Cu at (89.3, 87.8)
- added JP4: DMX_TX, Connector_PinHeader_1.00mm:PinHeader_1x03_P1.00mm_Horizontal, F.Cu at (147.5, 85.5)
- added U4: EEPROM-RP2040, WeAct-rp2040:WeAct-RP2040-Pico, F.Cu at (146.0, 62.8)
- U1: value rp2040-zero -> Controller-RP2040; footprint kleeb-mcu:rp2040-zero-smd -> WeAct-rp2040:WeAct-RP2040-Pico
- moved Address_16_OE1 46.8 mm to (130.5, 86.0), turned to 180 degrees
- moved Address_0_7 36.6 mm to (160.5, 62.5), turned to -90 degrees
- moved U1 14.0 mm to (145.9, 86.8)
- moved J1 4.94 mm to (170.2, 89.0)
- moved U2 4.94 mm to (160.0, 86.5)
Connections:
- U1 pad 1: unconnected-(U1-0-Pad1) -> /UART_EE_RX
- U1 pad 2: unconnected-(U1-1-Pad2) -> /UART_EE_TX
- U1 pad 22: /GND -> unconnected-(U1-GP19-Pad22)
- U1 pad 23: /VCC_5V -> /UART_ESP_RX
- U1 pad 6: unconnected-(U1-5-Pad6) -> /GND
- U2 pad 2: unconnected-(U2-~{RE}-Pad2) -> /VCC_5V
- U2 pad 3: unconnected-(U2-DE-Pad3) -> /VCC_5V
- U2 pad 4: unconnected-(U2-D-Pad4) -> /DMX_TX
- WIFI-ESP32C6 pad 12: unconnected-(WIFI-ESP32C6-3V3-Pad12) -> /VCC_3V3
- WIFI-ESP32C6 pad 7: unconnected-(WIFI-ESP32C6-PB08_A6_D6_TX-Pad7) -> /UART_ESP_TX
- WIFI-ESP32C6 pad 8: unconnected-(WIFI-ESP32C6-PB09_A7_D7_RX-Pad8) -> /UART_ESP_RX
Routing:
- net /VCC_5V: track 21.2 -> 214.6 mm, vias 0 -> 2
- net /VCC_3V3: track 0.00 -> 164.5 mm, vias 0 -> 8
- net /GND: track 137.3 -> 291.3 mm, vias 0 -> 3
- net /UART_EE_RX: track 0.00 -> 120.6 mm, vias 0 -> 5
- net /UART_EE_TX: track 0.00 -> 111.2 mm, vias 0 -> 3
- net /UART_ESP_TX: track 0.00 -> 84.2 mm
- net /UART_ESP_RX: track 0.00 -> 80.3 mm
- net /D7_3V3: track 0.00 -> 65.3 mm, vias 0 -> 1
- net /D6_3V3: track 0.00 -> 61.4 mm, vias 0 -> 1
- net /OE_3V3: track 0.00 -> 58.8 mm, vias 0 -> 1
- net /A8_3V3: track 0.00 -> 58.5 mm, vias 0 -> 2
- net /D5_3V3: track 0.00 -> 57.8 mm, vias 0 -> 1
- net /D4_3V3: track 0.00 -> 50.9 mm, vias 0 -> 1
- net /A0_5V: track 7.23 -> 54.7 mm, vias 0 -> 1
- net /D3_3V3: track 0.00 -> 47.2 mm, vias 0 -> 1
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