File: xiao-rp2040-probe/xiao-rp2040-probe.kicad_pcb (KiCad board)
At the start: 2 copper layers, 20 x 24 mm, 10 parts, among them J2 Conn_01x07_Pin, U1 MOUDLE-SEEEDUINO-XIAO

Commit message: Last pcb changes before order
Parts:
- J2: footprint Connector_PinHeader_2.54mm:PinHeader_1x07_P2.54mm_Horizontal -> Connector_PinHeader_2.54mm:PinHeader_1x07_P2.54mm_Vertical
- turned DAP_CONNECTED1 to 180 degrees
- turned DAP_TARGET_RUNNING1 to 180 degrees
- turned UART_RT1 to 180 degrees
- turned UART_TX1 to 180 degrees
Connections:
- DAP_CONNECTED1 pad 1: Net-(DAP_CONNECTED1-K) -> /GND
- DAP_CONNECTED1 pad 2: /3v3 -> Net-(DAP_CONNECTED1-A)
- DAP_TARGET_RUNNING1 pad 1: Net-(DAP_TARGET_RUNNING1-K) -> /GND
- DAP_TARGET_RUNNING1 pad 2: /3v3 -> Net-(DAP_TARGET_RUNNING1-A)
- J2 pad 1: /Ground -> /GND
- R1 pad 1: Net-(DAP_CONNECTED1-K) -> Net-(DAP_CONNECTED1-A)
- R2 pad 1: Net-(UART_RT1-K) -> Net-(UART_RT1-A)
- R3 pad 1: Net-(DAP_TARGET_RUNNING1-K) -> Net-(DAP_TARGET_RUNNING1-A)
- R4 pad 1: Net-(UART_TX1-K) -> Net-(UART_TX1-A)
- U1 pad 13: /Ground -> /GND
- UART_RT1 pad 1: Net-(UART_RT1-K) -> /GND
- UART_RT1 pad 2: /3v3 -> Net-(UART_RT1-A)
- UART_TX1 pad 1: Net-(UART_TX1-K) -> /GND
- UART_TX1 pad 2: /3v3 -> Net-(UART_TX1-A)
Routing:
- net /GND: track 0.00 -> 53.0 mm, vias 0 -> 5
- net /3v3: track 45.4 -> 22.0 mm, vias 2 -> 0
- net /Ground: track 17.8 -> 0.00 mm, vias 1 -> 0
- net Net-(UART_TX1-K): track 1.52 -> 0.00 mm
- net Net-(UART_TX1-A): track 0.00 -> 1.52 mm
- net Net-(UART_RT1-K): track 1.52 -> 0.00 mm
- net Net-(UART_RT1-A): track 0.00 -> 1.52 mm
- net Net-(DAP_TARGET_RUNNING1-K): track 1.52 -> 0.00 mm
- net Net-(DAP_TARGET_RUNNING1-A): track 0.00 -> 1.52 mm
- net Net-(DAP_CONNECTED1-K): track 1.52 -> 0.00 mm
- net Net-(DAP_CONNECTED1-A): track 0.00 -> 1.52 mm
- added copper zone on B.Cu, net /GND
- added copper zone on F.Cu, net /GND
Other:
- board text added: "2024-05-22 Jomer.dev"
- board text added: "XIAO-RP2040 Debug Probe Rev.1"
