File: xiao-rp2040-probe/xiao-rp2040-probe.kicad_sch (KiCad schematic)
At the start: 10 parts, among them J2 Conn_01x07_Pin, U1 MOUDLE-SEEEDUINO-XIAO

Commit message: Last pcb changes before order
Connections:
- net 3v3: no longer DAP_CONNECTED1.2 (A), DAP_TARGET_RUNNING1.2 (A), UART_RT1.2 (A), UART_TX1.2 (A)
- net at R4.1: now also UART_TX1.2 (A); no longer UART_TX1.1 (K)
- net at R3.1: now also DAP_TARGET_RUNNING1.2 (A); no longer DAP_TARGET_RUNNING1.1 (K)
- net at R1.1: now also DAP_CONNECTED1.2 (A); no longer DAP_CONNECTED1.1 (K)
- net at R2.1: now also UART_RT1.2 (A); no longer UART_RT1.1 (K)
- net Ground renamed GND
- net GND: now also DAP_CONNECTED1.1 (K), DAP_TARGET_RUNNING1.1 (K), UART_RT1.1 (K), UART_TX1.1 (K)
Other:
- moved on the sheet: DAP_CONNECTED1, DAP_TARGET_RUNNING1, UART_RT1, UART_TX1
Changed lines of the file:
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@@
 		)
 	)
-	(label "3v3"
+	(label "GND"
 		(at 82.55 88.9 0)
 		(fields_autoplaced yes)
@@
 		)
 	)
-	(label "3v3"
+	(label "GND"
 		(at 82.55 73.66 0)
 		(fields_autoplaced yes)
@@
 		)
 	)
-	(label "Ground"
+	(label "GND"
 		(at 139.7 102.87 0)
 		(fields_autoplaced yes)
@@
 		)
 	)
-	(label "3v3"
+	(label "GND"
 		(at 82.55 83.82 0)
 		(fields_autoplaced yes)
@@
 		)
 	)
-	(label "3v3"
+	(label "GND"
 		(at 82.55 78.74 0)
 		(fields_autoplaced yes)
@@
 	(symbol
 		(lib_id "Device:LED")
-		(at 92.71 78.74 180)
+		(at 92.71 78.74 0)
 		(unit 1)
 		(exclude_from_sim no)
@@
 		(dnp no)
 		(property "Reference" "UART_TX1"
-			(at 76.708 78.232 0)
+			(at 77.216 78.74 0)
 			(effects
 				(font
@@
 		)
 		(property "Value" "Red"
-			(at 89.408 79.756 0)
+			(at 96.012 77.724 0)
 			(effects
 				(font
@@
 	(symbol
 		(lib_id "Device:LED")
-		(at 92.71 88.9 180)
+		(at 92.71 88.9 0)
 		(unit 1)
 		(exclude_from_sim no)
@@
 		(dnp no)
 		(property "Reference" "DAP_CONNECTED1"
-			(at 73.914 88.646 0)
+			(at 74.168 88.9 0)
 			(effects
 				(font
@@
 		)
 		(property "Value" "Red"
-			(at 89.408 89.916 0)
+			(at 96.012 87.884 0)
 			(effects
 				(font
@@
 	(symbol
 		(lib_id "Device:LED")
-		(at 92.71 73.66 180)
+		(at 92.71 73.66 0)
 		(unit 1)
 		(exclude_from_sim no)
@@
 		(dnp no)
 		(property "Reference" "DAP_TARGET_RUNNING1"
-			(at 71.374 73.406 0)
+			(at 71.12 73.66 0)
 			(effects
 				(font
@@
 		)
 		(property "Value" "Red"
-			(at 89.408 74.676 0)
+			(at 96.012 72.644 0)
 			(effects
 				(font
@@
 	(symbol
 		(lib_id "Device:LED")
-		(at 92.71 83.82 180)
+		(at 92.71 83.82 0)
 		(unit 1)
 		(exclude_from_sim no)
@@
 		(dnp no)
 		(property "Reference" "UART_RT1"
-			(at 75.946 83.566 0)
+			(at 77.216 83.82 0)
 			(effects
 				(font
@@
 		)
 		(property "Value" "Red"
-			(at 89.408 84.836 0)
-			(effects
-				(font
+			(at 96.012 82.804 0)
+			(effects
+				(font
